File: mixing-board-jekyll/jekyll-one/jekyll-one.kicad_sch (KiCad schematic)
At the start: 25 parts, among them J1 Conn_01x04, J10 Conn_01x24, J11 Conn_01x05, J12 Conn_01x05, J2 Conn_01x04, J3 USB_C_Receptacle, J4 Conn_01x09, J5 Conn_01x05, J6 Conn_01x24, J7 Conn_01x04, J8 Conn_01x24_MountingPin, J9 Conn_01x24_MountingPin, P1 USB_C_Plug_USB2.0, SW1 SW_SPST, SW2 SW_SPST, SW3 SW_SPST, SW4 SW_SPST, U1 AMS1117-3.3, U2 ESP32-C3-MINI-1

Commit message: Use local thirdparty libraries.
Parts:
- J2: footprint (none) -> Connector_PinHeader_2.54mm:PinHeader_1x04_P2.54mm_Vertical
- J4: footprint (none) -> Connector_PinHeader_2.54mm:PinHeader_1x09_P2.54mm_Vertical
Changed lines of the file:
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@@
       (effects (font (size 1.27 1.27)) (justify left))
     )
-    (property "Footprint" "" (id 2) (at 69.85 160.02 0)
+    (property "Footprint" "Connector_PinHeader_2.54mm:PinHeader_1x09_P2.54mm_Vertical" (id 2) (at 69.85 160.02 0)
       (effects (font (size 1.27 1.27)) hide)
     )
@@
       (effects (font (size 1.27 1.27)) (justify left))
     )
-    (property "Footprint" "" (id 2) (at 30.48 176.53 0)
-      (effects (font (size 1.27 1.27)) hide)
-    )
+    (property "Footprint" "Connector_PinHeader_2.54mm:PinHeader_1x04_P2.54mm_Vertical" (id 2) (at 30.48 176.53 0)
+      (effects (font (size 1.27 1.27)) hide)
+    )
